Commit message: Обновил пакет с моделями робота и среды

File: object314_description/urdf/object314.xacro (robot description, xacro)
@@ -15,4 +15,5 @@
   <!-- Gazebo -->
   <xacro:include filename="$(find object314_description)/urdf/object314_gazebo.xacro"/>
+  <xacro:gazebo_plugin_p3d link="base_footprint"/>
   <!-- Base footprint size and position, m -->
   <xacro:property name="bf_length" value="1.323"/>

File: object314_description/urdf/object314_chassis.xacro (robot description, xacro)
@@ -52,5 +52,5 @@
         <origin xyz="0 0 0" rpy="${pi/2} 0 0"/>
         <geometry>
-          <cylinder radius="${w_radius}" length="${w_width}"/>
+          <cylinder radius="${w_radius}" length="${w_width/2}"/>
         </geometry>
       </collision>

File: object314_description/urdf/object314_gazebo.xacro (robot description, xacro)
@@ -42,4 +42,20 @@
         <kd value="1e6" />
         <fdir1 value="1 0 0"/>
+    </gazebo>
+  </xacro:macro>
+  <!-- Common plugins -->
+  <xacro:macro name="gazebo_plugin_p3d" params="link">
+    <gazebo>
+      <plugin name="gazebo_ros_p3d" filename="libgazebo_ros_p3d.so">
+        <ros>
+          <namespace></namespace>
+          <remapping>odom:=ground_truth</remapping>
+        </ros>
+        <body_name>${link}</body_name>
+        <update_rate>10</update_rate>
+        <xyz_offset>0 0 0</xyz_offset>
+        <rpy_offset>0 0 0</rpy_offset>
+        <gaussian_noise>0.00</gaussian_noise>
+      </plugin>
     </gazebo>
   </xacro:macro>
